File: AFE.sch (KiCad schematic (older format))
At the start: 28 parts, among them J3 JST PH SM4 S2B, J4 JST PH SM4 S2B, U2 INA317IDGKT, U3 INA317IDGKT, U4 OPA2349EA_250, U5 OPA2349EA_250

Commit message: redid power section with new energy harverster ic
Parts:
- renumbered C9 to C?, C15 to C?, C19 to C?, C17 to C?, C11 to C?, C8 to C?, C14 to C?, C18 to C?, C16 to C?, C10 to C?, J3 to J?, J4 to J?, R13 to R?, R15 to R?, R11 to R?, R9 to R?, R7 to R?, R12 to R?, R14 to R?, R10 to R?, R8 to R?, R6 to R?, TP16 to TP?, TP15 to TP?, U3 to U?, U5 to U?, U2 to U?, U4 to U?

Commit message: catch up
Parts:
- added C?: 0.1uF, Capacitor_SMD:C_0402_1005Metric, symbol Device:C_Small
- added FB?: 600 Ohm, symbol Device:Ferrite_Bead_Small
Connections:
- net VDDA: now also C?.1, FB?.1
- net GNDA renamed GND
- net GND: now also C?.2
- new net VDD: FB?.2
Changed lines of the file:
@@
-$EndComp
-$Comp
-L PatchV2:OPA2349EA_250 U?
-U 1 1 60558AF9
-P 5225 1750
-F 0 "U?" H 5750 2150 60  0000 C CNN
-F 1 "OPA2349EA_250" H 6025 1200 60  0000 C CNN
-F 2 "PatchV2:OPA2349EA" H 6045 2090 60  0001 C CNN
-F 3 "https://www.ti.com/lit/ds/symlink/opa2349.pdf?HQS=dis-dk-null-digikeymode-dsf-pf-null-wwe&ts=1616192746637" H 6025 2131 60  0001 C CNN
-	1    5225 1750
-	1    0    0    -1
 $EndComp
 $Comp
@@
 $EndComp
 Wire Wire Line
-	5225 1550 5050 1550
-Wire Wire Line
 	5050 1550 5050 1175
-Wire Wire Line
-	5050 1175 7025 1175
-Wire Wire Line
-	7025 1175 7025 1650
-Wire Wire Line
-	7025 1650 6825 1650
-Wire Wire Line
-	6125 875  7025 875
-Wire Wire Line
-	7025 875  7025 1175
-Connection ~ 7025 1175
 Wire Wire Line
 	5925 875  4325 875
@@
 Wire Wire Line
 	5025 2050 5025 2150
-Wire Wire Line
-	5025 2150 5225 2150
 Text Notes 8125 4050 0    75   ~ 0
 VDDA - 1.8V From power section LDO\nVCOM - 0.9V From power section LDO\nGNDA - GND for AFE and analog on uC, \n     join with GND near uC\n\nAll Rs 0.1% \nPlace deacap near each package\nSheild inputs with ground rail\nRemove ground plane from around INA gain resistor
@@
 $EndComp
 Wire Wire Line
-	5050 2650 5225 2650
-Wire Wire Line
 	5050 2525 5050 2650
 Wire Wire Line
@@
 $EndComp
 Wire Wire Line
-	5225 2850 5050 2850
-Wire Wire Line
 	5875 3275 5050 3275
 Wire Wire Line
@@
 Wire Wire Line
 	6950 2750 6825 2750
-$Comp
-L power:GNDA #PWR?
-U 1 1 6056C00B
-P 6925 2250
-F 0 "#PWR?" H 6925 2000 50  0001 C CNN
-F 1 "GNDA" H 6930 2077 50  0000 C CNN
-F 2 "" H 6925 2250 50  0001 C CNN
-F 3 "" H 6925 2250 50  0001 C CNN
-	1    6925 2250
-	1    0    0    -1
-$EndComp
-Wire Wire Line
-	6825 2150 6925 2150
-Wire Wire Line
-	6925 2150 6925 2250
 Wire Wire Line
 	6950 3275 6950 3500
@@
 Wire Wire Line
 	4250 1750 4325 1750
-Connection ~ 4775 1750
-Wire Wire Line
-	4775 1750 5225 1750
-Wire Wire Line
-	7025 1650 7275 1650
-Connection ~ 7025 1650
 Text HLabel 7275 1650 2    75   Output ~ 0
 AFE_CH1
@@
 	1    0    0    -1
 $EndComp
-$Comp
-L power:GNDA #PWR?
-U 1 1 60584069
-P 2650 2450
-F 0 "#PWR?" H 2650 2200 50  0001 C CNN
-F 1 "GNDA" H 2655 2277 50  0000 C CNN
-F 2 "" H 2650 2450 50  0001 C CNN
-F 3 "" H 2650 2450 50  0001 C CNN
-	1    2650 2450
-	1    0    0    -1
-$EndComp
-$Comp
-L power:GNDA #PWR?
-U 1 1 605849A7
-P 800 3500
-F 0 "#PWR?" H 800 3250 50  0001 C CNN
-F 1 "GNDA" H 805 3327 50  0000 C CNN
-F 2 "" H 800 3500 50  0001 C CNN
-F 3 "" H 800 3500 50  0001 C CNN
-	1    800  3500
-	1    0    0    -1
-$EndComp
 Wire Wire Line
 	800  3400 800  3450
@@
 Wire Wire Line
 	6925 5675 6800 5675
-$Comp
-L power:GNDA #PWR?
-U 1 1 605A1129
-P 6900 5175
-F 0 "#PWR?" H 6900 4925 50  0001 C CNN
-F 1 "GNDA" H 6905 5002 50  0000 C CNN
-F 2 "" H 6900 5175 50  0001 C CNN
-F 3 "" H 6900 5175 50  0001 C CNN
-	1    6900 5175
-	1    0    0    -1
-$EndComp
 Wire Wire Line
 	6800 5075 6900 5075
@@
 F 3 "~" H 1150 6225 50  0001 C CNN
 	1    1150 6225
-	1    0    0    -1
-$EndComp
-$Comp
-L power:GNDA #PWR?
-U 1 1 605A1186
-P 2625 5375
-F 0 "#PWR?" H 2625 5125 50  0001 C CNN
-F 1 "GNDA" H 2630 5202 50  0000 C CNN
-F 2 "" H 2625 5375 50  0001 C CNN
-F 3 "" H 2625 5375 50  0001 C CNN
-	1    2625 5375
-	1    0    0    -1
-$EndComp
-$Comp
-L power:GNDA #PWR?
-U 1 1 605A118C
-P 775 6425
-F 0 "#PWR?" H 775 6175 50  0001 C CNN
-F 1 "GNDA" H 780 6252 50  0000 C CNN
-F 2 "" H 775 6425 50  0001 C CNN
-F 3 "" H 775 6425 50  0001 C CNN
-	1    775  6425
 	1    0    0    -1
 $EndComp
@@
 $EndComp
 $Comp
-L power:GNDA #PWR?
-U 1 1 60ABEA96
+L power:GND #PWR?
+U 1 1 61737AA7
 P 1050 2400
 F 0 "#PWR?" H 1050 2150 50  0001 C CNN
-F 1 "GNDA" H 1055 2227 50  0000 C CNN
+F 1 "GND" H 1055 2227 50  0000 C CNN
 F 2 "" H 1050 2400 50  0001 C CNN
 F 3 "" H 1050 2400 50  0001 C CNN
@@
 $EndComp
 $Comp
-L power:GNDA #PWR?
-U 1 1 60ABEDB2
+L power:GND #PWR?
+U 1 1 61738138
+P 2650 2450
+F 0 "#PWR?" H 2650 2200 50  0001 C CNN
+F 1 "GND" H 2655 2277 50  0000 C CNN
+F 2 "" H 2650 2450 50  0001 C CNN
+F 3 "" H 2650 2450 50  0001 C CNN
+	1    2650 2450
+	1    0    0    -1
+$EndComp
+$Comp
+L power:GND #PWR?
+U 1 1 61738743
+P 6950 2250
+F 0 "#PWR?" H 6950 2000 50  0001 C CNN
+F 1 "GND" H 6955 2077 50  0000 C CNN
+F 2 "" H 6950 2250 50  0001 C CNN
+F 3 "" H 6950 2250 50  0001 C CNN
+	1    6950 2250
+	1    0    0    -1
+$EndComp
+Wire Wire Line
+	6125 875  7025 875
+Wire Wire Line
+	7025 875  7025 1175
+Wire Wire Line
+	5050 1175 7025 1175
+Connection ~ 7025 1650
+Connection ~ 7025 1175
+Wire Wire Line
+	7025 1175 7025 1650
+Wire Wire Line
+	7025 1650 6825 1650
+Wire Wire Line
+	7025 1650 7275 1650
+Connection ~ 4775 1750
+Wire Wire Line
+	5025 2150 5225 2150
+Wire Wire Line
+	5225 2850 5050 2850
+Wire Wire Line
+	5050 2650 5225 2650
+Wire Wire Line
+	4775 1750 5225 1750
+Wire Wire Line
+	5225 1550 5050 1550
+$Comp
+L PatchV2:OPA2349EA_250 U?
+U 1 1 60558AF9
+P 5225 1750
+F 0 "U?" H 5750 2150 60  0000 C CNN
+F 1 "OPA2349EA_250" H 6025 1200 60  0000 C CNN
+F 2 "PatchV2:OPA2349EA" H 6045 2090 60  0001 C CNN
+F 3 "https://www.ti.com/lit/ds/symlink/opa2349.pdf?HQS=dis-dk-null-digikeymode-dsf-pf-null-wwe&ts=1616192746637" H 6025 2131 60  0001 C CNN
+	1    5225 1750
+	1    0    0    -1
+$EndComp
+Wire Wire Line
+	6825 2150 6950 2150
+Wire Wire Line
+	6950 2150 6950 2250
+$Comp
+L power:GND #PWR?
+U 1 1 617654F8
+P 800 3500
+F 0 "#PWR?" H 800 3250 50  0001 C CNN
+F 1 "GND" H 805 3327 50  0000 C CNN
+F 2 "" H 800 3500 50  0001 C CNN
+F 3 "" H 800 3500 50  0001 C CNN
+	1    800  3500
+	1    0    0    -1
+$EndComp
+$Comp
+L power:GND #PWR?
+U 1 1 61765C3E
+P 775 6425
+F 0 "#PWR?" H 775 6175 50  0001 C CNN
+F 1 "GND" H 780 6252 50  0000 C CNN
+F 2 "" H 775 6425 50  0001 C CNN
+F 3 "" H 775 6425 50  0001 C CNN
+	1    775  6425
+	1    0    0    -1
+$EndComp
+$Comp
+L power:GND #PWR?
+U 1 1 61766D16
 P 1025 5325
 F 0 "#PWR?" H 1025 5075 50  0001 C CNN
-F 1 "GNDA" H 1030 5152 50  0000 C CNN
+F 1 "GND" H 1030 5152 50  0000 C CNN
 F 2 "" H 1025 5325 50  0001 C CNN
 F 3 "" H 1025 5325 50  0001 C CNN
@@
 	1    0    0    -1
 $EndComp
+$Comp
+L power:GND #PWR?
+U 1 1 61767134
+P 2625 5375
+F 0 "#PWR?" H 2625 5125 50  0001 C CNN
+F 1 "GND" H 2630 5202 50  0000 C CNN
+F 2 "" H 2625 5375 50  0001 C CNN
+F 3 "" H 2625 5375 50  0001 C CNN
+	1    2625 5375
+	1    0    0    -1
+$EndComp
+$Comp
+L power:GND #PWR?
+U 1 1 617674EA
+P 6900 5175
+F 0 "#PWR?" H 6900 4925 50  0001 C CNN
+F 1 "GND" H 6905 5002 50  0000 C CNN
+F 2 "" H 6900 5175 50  0001 C CNN
+F 3 "" H 6900 5175 50  0001 C CNN
+	1    6900 5175
+	1    0    0    -1
+$EndComp
+$Comp
+L Device:C_Small C?
+U 1 1 617737FD
+P 2425 7200
+F 0 "C?" H 2517 7246 50  0000 L CNN
+F 1 "0.1uF" H 2517 7155 50  0000 L CNN
+F 2 "Capacitor_SMD:C_0402_1005Metric" H 2425 7200 50  0001 C CNN
+F 3 "~" H 2425 7200 50  0001 C CNN
+	1    2425 7200
+	1    0    0    -1
+$EndComp
+Wire Wire Line
+	2425 7050 2425 7100
+$Comp
+L power:GND #PWR?
+U 1 1 617893F1
+P 2425 7400
+F 0 "#PWR?" H 2425 7150 50  0001 C CNN
+F 1 "GND" H 2430 7227 50  0000 C CNN
+F 2 "" H 2425 7400 50  0001 C CNN
+F 3 "" H 2425 7400 50  0001 C CNN
+	1    2425 7400
+	1    0    0    -1
+$EndComp
+Wire Wire Line
+	2425 7300 2425 7400
+$Comp
+L power:VDDA #PWR?
+U 1 1 6178ECF5
+P 2425 6950
+F 0 "#PWR?" H 2425 6800 50  0001 C CNN
+F 1 "VDDA" H 2440 7123 50  0000 C CNN
+F 2 "" H 2425 6950 50  0001 C CNN
+F 3 "" H 2425 6950 50  0001 C CNN
+	1    2425 6950
+	1    0    0    -1
+$EndComp
+Wire Wire Line
+	2425 6950 2425 7050
+Connection ~ 2425 7050
+$Comp
+L power:VDD #PWR?
+U 1 1 61793D2C
+P 1725 6950
+F 0 "#PWR?" H 1725 6800 50  0001 C CNN
+F 1 "VDD" H 1740 7123 50  0000 C CNN
+F 2 "" H 1725 6950 50  0001 C CNN
+F 3 "" H 1725 6950 50  0001 C CNN
+	1    1725 6950
+	1    0    0    -1
+$EndComp
+Wire Wire Line
+	1725 7050 1725 6950
+Wire Wire Line
+	1725 7050 1975 7050
+Wire Wire Line
+	2175 7050 2425 7050
+$Comp
+L Device:Ferrite_Bead_Small FB?
+U 1 1 61774673
+P 2075 7050
+F 0 "FB?" V 1838 7050 50  0000 C CNN
+F 1 "600 Ohm" V 1929 7050 50  0000 C CNN
+F 2 "" V 2005 7050 50  0001 C CNN
+F 3 "~" H 2075 7050 50  0001 C CNN
+F 4 "490-1006-1-ND" V 2075 7050 50  0001 C CNN "DigiKey_PN"
+	1    2075 7050
+	0    1    1    0
+$EndComp
 $EndSCHEMATC

Commit message: schematic functionally finished working on layout
Parts:
- removed C? (x2): 0.1uF, Capacitor_SMD:C_0402_1005Metric, symbol Device:C_Small
- removed R? (x2): 5.23k 0.1%, Resistor_SMD:R_0402_1005Metric, symbol Device:R
- removed U? (x2): INA317IDGKT, PatchV2:INA317IDGKT, symbol PatchV2:INA317IDGKT
- added C8: 0.1uF, Capacitor_SMD:C_0402_1005Metric, symbol Device:C_Small
- added R10, R9: 10k 0.1%, Resistor_SMD:R_0402_1005Metric, symbol Device:R
- added R11, R12: 90.9k 0.1%, Resistor_SMD:R_0402_1005Metric, symbol Device:R
- added U2: INA2321EA_250, PatchV2:INA2321EA&slash_250, symbol PatchV2:INA2321EA_250
- FB1: renamed from FB?; footprint (none) -> Inductor_SMD:L_0402_1005Metric
- gave numbers to parts that had none: 23
Connections:
- net GND: now also C8.2, U2.4 (V-)
- net VCOM: now also U2.2 (VIN-A), U2.6 (VIN-B)
- net VDDA: now also C8.1, U2.11 (V+)
- net at J6.2 (Pin_2), R8.2: now also U2.3 (VIN+A)
- net REFA: now reaches C13.1, U4.7 (OUTB)
- net REFA: now also R9.2, U2.12 (REFA)
- net at R14.2, R16.2, TP6.1: now also R11.1, U2.13 (VOUTA)
- net at J5.2 (Pin_2), R7.2: now also U2.5 (VIN+B)
- net REFB: now reaches C12.1, U3.7 (OUTB)
- net REFB: now also R10.2, U2.10 (REFB)
- net at R13.2, R15.2, TP5.1: now also R12.1, U2.9 (VOUTB)
- new net: R11.2, R9.1, U2.1 (RGA)
- new net: R10.1, R12.2, U2.7 (RGB)
- no-connect marks 0 -> 2
Other:
- moved on the sheet: C10, C11, C12, C13, C14, C15, C9, FB1, J5, J6, R13, R14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

Commit message: Finished pre-review layout
Parts:
- added C24: 0.1uF, Capacitor_SMD:C_0402_1005Metric, symbol Device:C_Small
Connections:
- net AFE_CH1: now also C14.1, U3.1 (OUTA), U3.2 (INA-); no longer C15.1, U4.1 (OUTA), U4.2 (INA-)
- net AFE_CH2: now also C15.1, U4.1 (OUTA), U4.2 (INA-); no longer C14.1, U3.1 (OUTA), U3.2 (INA-)
- net GND: now also C24.2
- net VDD: now also C24.1
- net at R8.2, U2.3 (VIN+A): now also J5.2 (Pin_2); no longer J6.2 (Pin_2)
- net at R7.2, U2.5 (VIN+B): now also J6.2 (Pin_2); no longer J5.2 (Pin_2)
Other:
- moved on the sheet: J5, J6
Changed lines of the file:
@@
 Wire Wire Line
 	7350 1675 7425 1675
-Text HLabel 10375 1575 2    75   Output ~ 0
+Text HLabel 10350 4500 2    75   Output ~ 0
 AFE_CH1
 $Comp
@@
 	-1   0    0    1
 $EndComp
-Connection ~ 1900 2625
-Wire Wire Line
-	1175 2625 1900 2625
-Wire Wire Line
-	1175 2725 1300 2725
-Wire Wire Line
-	1300 2725 1300 2875
+Wire Wire Line
+	1150 3825 1875 3825
+Wire Wire Line
+	1150 3925 1275 3925
+Wire Wire Line
+	1275 3925 1275 4075
 $Comp
 L PatchV2:OPA2349EA_250 U3
@@
 	10100 4500 10350 4500
 Connection ~ 10100 4500
-Text HLabel 10350 4500 2    75   Output ~ 0
+Text HLabel 10375 1575 2    75   Output ~ 0
 AFE_CH2
 $Comp
@@
 L Connector_Generic:Conn_01x02 J5
 U 1 1 605A1162
-P 950 3925
-F 0 "J5" H 868 3600 50  0000 C CNN
-F 1 "JST PH SM4 S2B" H 850 3700 50  0000 C CNN
-F 2 "PatchV2:JST-S2B-PH-SM4-TBLFSN-Manufacturer_Recommended" H 950 3925 50  0001 C CNN
-F 3 "~" H 950 3925 50  0001 C CNN
-	1    950  3925
-	-1   0    0    1
-$EndComp
-Wire Wire Line
-	1150 3825 1875 3825
-Wire Wire Line
-	1150 3925 1275 3925
-Wire Wire Line
-	1275 3925 1275 4075
+P 975 2725
+F 0 "J5" H 893 2400 50  0000 C CNN
+F 1 "JST PH SM4 S2B" H 875 2500 50  0000 C CNN
+F 2 "PatchV2:JST-S2B-PH-SM4-TBLFSN-Manufacturer_Recommended" H 975 2725 50  0001 C CNN
+F 3 "~" H 975 2725 50  0001 C CNN
+	1    975  2725
+	-1   0    0    1
+$EndComp
+Wire Wire Line
+	1175 2625 1900 2625
+Wire Wire Line
+	1175 2725 1300 2725
+Wire Wire Line
+	1300 2725 1300 2875
 Wire Wire Line
 	775  6325 775  6375
@@
 L Connector_Generic:Conn_01x02 J6
 U 1 1 6096A277
-P 975 2725
-F 0 "J6" H 893 2400 50  0000 C CNN
-F 1 "JST PH SM4 S2B" H 875 2500 50  0000 C CNN
-F 2 "PatchV2:JST-S2B-PH-SM4-TBLFSN-Manufacturer_Recommended" H 975 2725 50  0001 C CNN
-F 3 "~" H 975 2725 50  0001 C CNN
-	1    975  2725
+P 950 3925
+F 0 "J6" H 868 3600 50  0000 C CNN
+F 1 "JST PH SM4 S2B" H 850 3700 50  0000 C CNN
+F 2 "PatchV2:JST-S2B-PH-SM4-TBLFSN-Manufacturer_Recommended" H 950 3925 50  0001 C CNN
+F 3 "~" H 950 3925 50  0001 C CNN
+	1    950  3925
 	-1   0    0    1
 $EndComp
@@
 L power:GND #PWR0135
 U 1 1 61737AA7
-P 1300 2875
-F 0 "#PWR0135" H 1300 2625 50  0001 C CNN
-F 1 "GND" H 1305 2702 50  0000 C CNN
-F 2 "" H 1300 2875 50  0001 C CNN
-F 3 "" H 1300 2875 50  0001 C CNN
-	1    1300 2875
+P 1275 4075
+F 0 "#PWR0135" H 1275 3825 50  0001 C CNN
+F 1 "GND" H 1280 3902 50  0000 C CNN
+F 2 "" H 1275 4075 50  0001 C CNN
+F 3 "" H 1275 4075 50  0001 C CNN
+	1    1275 4075
 	1    0    0    -1
 $EndComp
@@
 L power:GND #PWR0138
 U 1 1 61766D16
-P 1275 4075
-F 0 "#PWR0138" H 1275 3825 50  0001 C CNN
-F 1 "GND" H 1280 3902 50  0000 C CNN
-F 2 "" H 1275 4075 50  0001 C CNN
-F 3 "" H 1275 4075 50  0001 C CNN
-	1    1275 4075
+P 1300 2875
+F 0 "#PWR0138" H 1300 2625 50  0001 C CNN
+F 1 "GND" H 1305 2702 50  0000 C CNN
+F 2 "" H 1300 2875 50  0001 C CNN
+F 3 "" H 1300 2875 50  0001 C CNN
+	1    1300 2875
 	1    0    0    -1
 $EndComp
@@
 Wire Wire Line
 	2450 2625 2450 3225
+Wire Wire Line
+	1875 3825 3125 3825
+Wire Wire Line
+	2450 3225 3125 3225
+Connection ~ 1900 2625
 Connection ~ 1875 3825
-Wire Wire Line
-	1875 3825 3125 3825
-Wire Wire Line
-	2450 3225 3125 3225
+$Comp
+L Device:C_Small C24
+U 1 1 6164D3E0
+P 2600 6200
+F 0 "C24" H 2692 6246 50  0000 L CNN
+F 1 "0.1uF" H 2692 6155 50  0000 L CNN
+F 2 "Capacitor_SMD:C_0402_1005Metric" H 2600 6200 50  0001 C CNN
+F 3 "~" H 2600 6200 50  0001 C CNN
+	1    2600 6200
+	1    0    0    -1
+$EndComp
+Wire Wire Line
+	2600 6100 2600 6025
+Connection ~ 2600 6025
+$Comp
+L power:GND #PWR0150
+U 1 1 61653D18
+P 2600 6400
+F 0 "#PWR0150" H 2600 6150 50  0001 C CNN
+F 1 "GND" H 2605 6227 50  0000 C CNN
+F 2 "" H 2600 6400 50  0001 C CNN
+F 3 "" H 2600 6400 50  0001 C CNN
+	1    2600 6400
+	1    0    0    -1
+$EndComp
+Wire Wire Line
+	2600 6300 2600 6400
 $EndSCHEMATC
